Commit message: caster_steering

File: vehicle/xacro/ai_car1.xacro (robot description, xacro)
@@ -47,5 +47,5 @@
     caster_back="${CASTER_BACK}" parent="${BASE}"
     x="-0.76" y="0.0" z="${CASTER_RADIUS}"
-    roll="${90.0*D2R}" pitch="0.0" yaw="${90.0*D2R}"/>
+    roll="0.0" pitch="0.0" yaw="0.0"/>
   <xacro:caster_back_link_macro
     caster_back="${CASTER_BACK}"

File: vehicle/xacro/parts/caster_back_macro.xacro (robot description, xacro)
@@ -1,12 +1,19 @@
 <?xml version="1.0" ?>
 <robot xmlns:xacro="http://www.ros.org/wiki/xacro">
+  <xacro:property name="PI" value="3.1415926"/>
   <xacro:macro name="caster_back_joint_macro"
                params="caster_back parent
                        x y z roll pitch yaw">
+    <joint name="${caster_back}_steering_joint" type="continuous">
+      <parent link="${parent}_link"/>
+      <child  link="${caster_back}_steering_link"/>
+      <origin xyz="${x} ${y} ${z}" rpy="${roll} ${pitch} ${yaw}"/>
+      <axis xyz="0 0 1"/>
+    </joint>
     <joint name="${caster_back}_joint" type="continuous">
-      <parent link="${parent}_link"/>
+      <parent link="${caster_back}_steering_link"/>
       <child  link="${caster_back}_link"/>
-      <origin xyz="${x} ${y} ${z}" rpy="${roll} ${pitch} ${yaw}"/>
-      <axis xyz="1 0 0"/>
+      <origin xyz="-0.2 0 0" rpy="0 0 0"/>
+      <axis xyz="0 1 0"/>
     </joint>
   </xacro:macro>
@@ -16,7 +23,8 @@
     <xacro:property name="MESH_FILE" value="package://vehicle/xacro/meshes/tire.dae"/>
     <xacro:property name="SCALE" value="0.10"/>
+    <link name="${caster_back}_steering_link"/>
     <link name="${caster_back}_link">
       <visual>
-        <origin xyz="${x} ${y} ${z}" rpy="${roll} ${pitch} ${yaw}"/>
+        <origin xyz="${x} ${y} ${z}" rpy="${roll} ${pitch} ${yaw+PI/2}"/>
         <geometry>
           <mesh filename="${MESH_FILE}" scale="${SCALE} ${SCALE} ${SCALE}"/>
@@ -24,5 +32,5 @@
       </visual>
       <collision>
-        <origin xyz="${x} ${y} ${z}" rpy="${roll} ${pitch} ${yaw}"/>
+        <origin xyz="${x} ${y} ${z}" rpy="${roll} ${pitch} ${yaw+PI/2}"/>
         <geometry>
           <mesh filename="${MESH_FILE}" scale="${SCALE} ${SCALE} ${SCALE}"/>
@@ -34,5 +42,5 @@
       </collision>
       <inertial>
-        <origin xyz="${x} ${y} ${z}" rpy="${roll} ${pitch} ${yaw}"/>
+        <origin xyz="${x} ${y} ${z}" rpy="${roll} ${pitch} ${yaw+PI/2}"/>
         <mass value="0.005" />
         <inertia ixx="0.001" ixy="0.0" ixz="0.0" iyy="0.001" iyz="0.0" izz="0.001"/>
