Commit message: fixed get sample_vehielce package

File: vehicles/sample_vehicle/xacro/parts/base_macro.xacro (robot description, xacro)
@@ -9,5 +9,5 @@
       <origin xyz="0.0  0.0  0.0" rpy="0.0  0.0  0.0"/>
     </joint>
-    <xacro:property name="MESH_FILE" value="package://vehicle/xacro/meshes/AIF_body.dae"/>
+    <xacro:property name="MESH_FILE" value="package://sample_vehicle/xacro/meshes/AIF_body.dae"/>
     <link name="${base}_link">
       <visual>

File: vehicles/sample_vehicle/xacro/parts/caster_back_macro.xacro (robot description, xacro)
@@ -14,5 +14,5 @@
                params="caster_back
                        x y z roll pitch yaw">
-    <xacro:property name="MESH_FILE" value="package://vehicle/xacro/meshes/tire.dae"/>
+    <xacro:property name="MESH_FILE" value="package://sample_vehicle/xacro/meshes/tire.dae"/>
     <xacro:property name="SCALE" value="0.10"/>
     <link name="${caster_back}_link">

File: vehicles/sample_vehicle/xacro/parts/wheel_macro.xacro (robot description, xacro)
@@ -14,5 +14,5 @@
                params="wheel
                        x y z roll pitch yaw">
-    <xacro:property name="MESH_FILE" value="package://vehicle/xacro/meshes/tire.dae"/>
+    <xacro:property name="MESH_FILE" value="package://sample_vehicle/xacro/meshes/tire.dae"/>
     <xacro:property name="THICKNESS_SCALE" value="0.05"/>
     <xacro:property name="SIZE_SCALE" value="0.12"/>

File: vehicles/sample_vehicle/xacro/parts/zed_macro.xacro (robot description, xacro)
@@ -3,8 +3,8 @@
   <xacro:macro name="zed_macro"
                params="camera parent">
-    <xacro:property name="ZED_PARAM_YAML_PATH" value="$(find vehicle)/config/zedx/extrinsic/extrinsic.yaml" />
+    <xacro:property name="ZED_PARAM_YAML_PATH" value="$(find sample_vehicle)/config/zedx/extrinsic/extrinsic.yaml" />
     <xacro:property name="POSITION" value="${load_yaml(ZED_PARAM_YAML_PATH)['position']}" />
     <xacro:property name="ORIENTATION" value="${load_yaml(ZED_PARAM_YAML_PATH)['orientation']}" />
-    <xacro:property name="MESH_FILE" value="package://vehicle/xacro/meshes/zedx.stl"/>
+    <xacro:property name="MESH_FILE" value="package://sample_vehicle/xacro/meshes/zedx.stl"/>
     <xacro:property name="SIZE" value="${dict(x=0.035, y=0.16, z=0.03)}"/>
     <xacro:property name="BASE_LINE" value="0.120005"/>
